File: Графические материалы/thermal_imager/thermal_imager.kicad_pcb (KiCad board)
At the start: 2 copper layers, 57.2 x 38.1 mm, 24 parts

Commit message: Плакаты готовы
Parts:
- added XS2: SWD, Connector_PinSocket_1.00mm:PinSocket_1x04_P1.00mm_Vertical, F.Cu at (130.3, 152.1)
- turned XS1 to 90 degrees
Connections:
- XS1 pad 6: GND -> (no net)
Routing:
- net Net-(DD3-Pad46): track 0.00 -> 36.1 mm
- net Net-(DD3-Pad22): track 33.8 -> 9.72 mm
- net Net-(DD3-Pad23): track 9.48 -> 28.0 mm
- net Net-(DD3-Pad20): track 32.9 -> 15.1 mm
- net Net-(DD3-Pad49): track 0.00 -> 13.4 mm
- net Net-(BK1-Pad4): track 26.9 -> 15.1 mm
- net Net-(BK1-Pad1): track 16.6 -> 13.7 mm
- net Net-(C1-Pad2): track 37.0 -> 39.2 mm
- net GND: track 135.4 -> 137.3 mm
